Commit message: Cleaned up file and made variables

File: helios/description/sensors.xacro (robot description, xacro)
@@ -1,13 +1,15 @@
 <?xml version="1.0"?>
 <robot xmlns:xacro="http://www.ros.org/wiki/xacro" name="helios">
+    <!-- ZED2i and Camera Pole ======================================================== -->
+    <!-- Camera Pole Properties -->
     <xacro:property name="camera_pole_width" value="0.03"/>
     <xacro:property name="camera_pole_height" value="0.6"/>
     <xacro:property name="camera_pole_mass" value="0.01"/>
+    <!-- ZED2i Camera Properties -->
     <xacro:property name="zed2i_length" value="0.28"/>
     <xacro:property name="zed2i_width" value="0.03"/>
     <xacro:property name="zed2i_height" value="0.03"/>
     <xacro:property name="zed2i_mass" value="0.01"/>
-    <!-- CAMERA LINK -->
-    <!-- camera pole -->
+    <!-- camera pole joint -->
     <joint name="camera_pole_joint" type="fixed">
         <parent link="chassis_link"/>
@@ -15,4 +17,5 @@
         <origin xyz="${camera_pole_width/2} 0 ${chassis_height}"/>
     </joint>
+    <!-- camera pole link -->
     <link name="camera_pole_link">
         <visual>
@@ -33,5 +36,5 @@
         </xacro:inertial_box>
     </link>
-    <!-- zed2i camera -->
+    <!-- zed2i camera joint -->
     <joint name="zed2i_joint" type="fixed">
         <parent link="camera_pole_link"/>
@@ -39,4 +42,5 @@
         <origin xyz="0 0 ${camera_pole_height}"/>
     </joint>
+    <!-- zed2i camera link -->
     <link name="zed2i_link">
         <visual>
@@ -57,18 +61,23 @@
         </xacro:inertial_box>
     </link>
-    <!-- LIDAR  -->
-    <!-- Lidar Joint -->
+    <!-- LIDAR ======================================================== -->
+    <!-- TODO - Update property values to be correct -->
+    <!-- LIDAR Properties -->
+    <xacro:property name="lidar_height" value="0.03"/>
+    <xacro:property name="lidar_radius" value="0.03"/>
+    <xacro:property name="lidar_mass" value="0.01"/>
+    <!-- LIDAR Joint -->
     <joint name="lidar_joint" type="fixed">
         <axis xyz="0 1 0" />
-        <origin xyz="0 3 0" rpy="0 0 0"/>
+        <origin xyz="0 0 1" rpy="0 0 0"/>
         <parent link="chassis_link"/>
         <child link="lidar_link"/>
     </joint>
-    <!-- Lidar Link -->
+    <!-- LIDAR Link -->
     <link name="lidar_link">
         <collision>
             <origin xyz="0 0 0" rpy="0 0 0"/>
             <geometry>
-                <box size="0.1 0.1 0.1"/>
+                <cylinder length="${lidar_height}" radius="${lidar_radius}"/>
             </geometry>
         </collision>
@@ -76,13 +85,10 @@
             <origin xyz="0 0 0" rpy="0 0 0"/>
             <geometry>
-                <box size="0.1 0.1 0.1"/>
+                <cylinder length="${lidar_height}" radius="${lidar_radius}"/>
             </geometry>
         </visual>
-        <!-- ToDO replace this -->
-        <inertial>
-            <mass value="1e-5" />
+        <xacro:inertial_cylinder mass="${lidar_mass}" length="${lidar_height}" radius="${lidar_radius}">
             <origin xyz="0 0 0" rpy="0 0 0"/>
-            <inertia ixx="1e-6" ixy="0" ixz="0" iyy="1e-6" iyz="0" izz="1e-6" />
-        </inertial>
+        </xacro:inertial_cylinder>
     </link>
 </robot>
