Commit message: added ros2_control support with keyboard

File: helios/description/robot.urdf.xacro (robot description, xacro)
@@ -4,5 +4,4 @@
     <xacro:include filename="sensors.xacro"/>
     <xacro:include filename="gazebo.xacro"/>
-    <!-- <xacro:include filename="ros2_control.xacro"/> -->
-    <!-- <xacro:include filename="lidar.xacro"/> -->
+    <xacro:include filename="ros2_control.xacro"/>
 </robot>

File: helios/description/ros2_control.xacro (robot description, xacro)
@@ -1,13 +1,13 @@
 <?xml version="1.0"?>
 <robot xmlns:xacro="http://www.ros.org/wiki/xacro">
-    <xacro:property name="min_vel" value="-10"/>
-    <xacro:property name="max_vel" value="10"/>
+    <!-- <xacro:property name="min_vel" value="-10"/>
+    <xacro:property name="max_vel" value="10"/> -->
     <!-- hardware interface for controller manager -->
     <ros2_control name="GazeboSystem" type="system">
         <hardware>
-            <!-- change to work with ignition-->
             <plugin>gazebo_ros2_control/GazeboSystem</plugin>
         </hardware>
-        <!-- LEFT WHEEL -->
+        <!-- LEFT WHEELS -->
+        <!-- front left wheel -->
         <joint name="front_left_wheel_joint">
             <command_interface name="velocity">
@@ -18,6 +18,25 @@
             <state_interface name="position"/>
         </joint>
-        <!-- RIGHT WHEEL -->
+        <!-- back left wheel -->
+        <joint name="back_left_wheel_joint">
+            <command_interface name="velocity">
+                <param name="min">-10</param>
+                <param name="max">10</param>
+            </command_interface>
+            <state_interface name="velocity"/>
+            <state_interface name="position"/>
+        </joint>
+        <!-- RIGHT WHEELS -->
+        <!-- front right wheel -->
         <joint name="front_right_wheel_joint">
+            <command_interface name="velocity">
+                <param name="min">-10</param>
+                <param name="max">10</param>
+            </command_interface>
+            <state_interface name="velocity"/>
+            <state_interface name="position"/>
+        </joint>
+        <!-- back right wheel -->
+        <joint name="back_right_wheel_joint">
             <command_interface name="velocity">
                 <param name="min">-10</param>
@@ -32,7 +51,6 @@
     <!-- ros2 run controller_manager ros2_control_node -->
     <gazebo>
-        <!-- change to work with ignition-->
         <plugin name="gazebo_ros2_control" filename="libgazebo_ros2_control.so">
-            <parameters>$(find helios)/confog/my_controllers.yaml</parameters>
+            <parameters>$(find helios)/config/my_controllers.yaml</parameters>
         </plugin>
     </gazebo>
