Commit message: added camera support

File: helios/description/chassis.xacro (robot description, xacro)
@@ -21,8 +21,8 @@
     <joint name="chassis_joint" type="fixed">
         <parent link="base_link"/>
-        <child link="chassis"/>
+        <child link="chassis_link"/>
         <origin xyz="${-chassis_length/2} 0 0"/>
     </joint>
-    <link name="chassis">
+    <link name="chassis_link">
         <visual>
             <origin xyz="${chassis_length/2} 0 ${chassis_height/2}"/>
@@ -46,9 +46,9 @@
     <joint name="front_left_wheel_joint" type="continuous">
         <parent link="base_link"/>
-        <child link="front_left_wheel"/>
+        <child link="front_left_wheel_link"/>
         <origin xyz="${wheel_dist_from_center} ${chassis_width/2 + wheel_width/2} 0" rpy="${-pi/2} 0 0"/>
         <axis xyz="0 0 1"/>
     </joint>
-    <link name="front_left_wheel">
+    <link name="front_left_wheel_link">
         <visual>
             <geometry>
@@ -69,9 +69,9 @@
     <joint name="back_left_wheel_joint" type="continuous">
         <parent link="base_link"/>
-        <child link="back_left_wheel"/>
+        <child link="back_left_wheel_link"/>
         <origin xyz="${-wheel_dist_from_center} ${chassis_width/2 + wheel_width/2} 0" rpy="${-pi/2} 0 0"/>
         <axis xyz="0 0 1"/>
     </joint>
-    <link name="back_left_wheel">
+    <link name="back_left_wheel_link">
         <visual>
             <geometry>
@@ -93,9 +93,9 @@
     <joint name="front_right_wheel_joint" type="continuous">
         <parent link="base_link"/>
-        <child link="front_right_wheel"/>
+        <child link="front_right_wheel_link"/>
         <origin xyz="${wheel_dist_from_center} ${-(chassis_width/2 + wheel_width/2)} 0" rpy="${pi/2} 0 0"/>
         <axis xyz="0 0 -1"/>
     </joint>
-    <link name="front_right_wheel">
+    <link name="front_right_wheel_link">
         <visual>
             <geometry>
@@ -116,9 +116,9 @@
     <joint name="back_right_wheel_joint" type="continuous">
         <parent link="base_link"/>
-        <child link="back_right_wheel"/>
+        <child link="back_right_wheel_link"/>
         <origin xyz="${-wheel_dist_from_center} ${-(chassis_width/2 + wheel_width/2)} 0" rpy="${pi/2} 0 0"/>
         <axis xyz="0 0 -1"/>
     </joint>
-    <link name="back_right_wheel">
+    <link name="back_right_wheel_link">
         <visual>
             <geometry>

File: helios/description/gazebo.xacro (robot description, xacro)
@@ -4,15 +4,21 @@
         <material>Gazebo/White</material>
     </gazebo>
-    <gazebo reference="front_left_wheel">
+    <gazebo reference="front_left_wheel_link">
         <material>Gazebo/Blue</material>
     </gazebo>
-        <gazebo reference="front_right_wheel">
+    <gazebo reference="front_right_wheel_link">
         <material>Gazebo/Blue</material>
     </gazebo>
-        <gazebo reference="back_left_wheel">
+    <gazebo reference="back_left_wheel_link">
         <material>Gazebo/Blue</material>
     </gazebo>
-        <gazebo reference="back_right_wheel">
+    <gazebo reference="back_right_wheel_link">
         <material>Gazebo/Blue</material>
+    </gazebo>
+    <gazebo reference="camera_pole_link">
+        <material>Gazebo/Red</material>
+    </gazebo>
+    <gazebo reference="zed2i_link">
+        <material>Gazebo/Black</material>
     </gazebo>
     <!-- TODO change later to use gazebo_ros_control plugin instead -->
@@ -28,13 +34,13 @@
     </gazebo>
     <!-- create link and joint for optical camera frame -->
-    <!-- <joint name="camera_optical_joint" type="fixed">
+    <joint name="zed2i_optical_joint" type="fixed">
         <origin xyz = "0 0 0" rpy="-1.571 0 -1.571"/>
-        <parent link="camera_link"/>
-        <child link="camera_link_opical"/>
+        <parent link="zed2i_link"/>
+        <child link="zed2i_link_optical"/>
     </joint>
-    <link name="camera_link_optical"></link> -->
+    <link name="zed2i_link_optical"></link>
     <!-- add gazebo setup for camera-->
-    <!-- <gazebo reference="camera_link">
-        <sensor type="depth" name="zed2i">
+    <gazebo reference="zed2i_link">
+        <sensor type="camera" name="zed2i">
             <update_rate>20</update_rate>
             <visualize>true</visualize>
@@ -57,5 +63,9 @@
             </camera>
             <plugin name="camera_controller" filename="libgazebo_ros_camera.so">
+                <frame_name>camera_link_optical</frame_name>
+                <min_depth>0.1</min_depth>
+                <max_depth>500</max_depth>
+            </plugin>
         </sensor>
-    </gazebo> -->
+    </gazebo>
 </robot>

File: helios/description/robot.urdf.xacro (robot description, xacro)
@@ -1,5 +1,6 @@
 <?xml version="1.0"?>
 <robot xmlns:xacro="http://www.ros.org/wiki/xacro" name="helios">
-    <xacro:include filename="robot_core.xacro"/>
+    <xacro:include filename="chassis.xacro"/>
+    <xacro:include filename="sensors.xacro"/>
     <xacro:include filename="gazebo.xacro"/>
     <!-- <xacro:include filename="ros2_control.xacro"/> -->

Commit message: added SLAM setup, visualize launch file

File: helios/description/chassis.xacro (robot description, xacro)
@@ -16,4 +16,12 @@
     <!-- Base link sits at bottom center of chassis -->
     <link name="base_link">
+    </link>
+    <!-- BASE_FOOTPRINT_LINK -->
+    <joint name="base_footprint_joint" type="fixed">
+        <parent link="base_link"/>
+        <child link="base_footprint_link"/>
+        <origin xyz="0 0 0" rpy="0 0 0"/>
+    </joint>
+    <link name="base_footprint_link">
     </link>
     <!-- CHASSIS LINK -->

File: helios/description/sensors.xacro (robot description, xacro)
@@ -32,5 +32,5 @@
             </geometry>
         </collision>
-        <xacro:inertial_box mass="${camera_pole_mass}" x="0" y="0" z="${camera_pole_height/2}">
+        <xacro:inertial_box mass="${camera_pole_mass}" x="${camera_pole_width}" y="${camera_pole_width}" z="${camera_pole_height}">
             <origin xyz="0 0 ${camera_pole_height/2}" rpy="0 0 0"/>
         </xacro:inertial_box>
@@ -57,5 +57,5 @@
             </geometry>
         </collision>
-        <xacro:inertial_box mass="${zed2i_mass}" x="0" y="0" z="${zed2i_height/2}">
+        <xacro:inertial_box mass="${zed2i_mass}" x="${zed2i_width}" y="${zed2i_length}" z="${zed2i_height}">
             <origin xyz="0 0 ${zed2i_height/2}" rpy="0 0 0"/>
         </xacro:inertial_box>
