Commit message: Added to URDF

File: helios/description/gazebo.xacro (robot description, xacro)
@@ -1,3 +1,46 @@
 <?xml version="1.0"?>
 <robot xmlns:xacro="http://www.ros.org/wiki/xacro">]
+    <!-- TODO change later to use gazebo_ros_control plugin instead -->
+    <gazebo>
+        <plugin name="gazebo_ros_joint_state_publisher"
+            filename="libgazebo_ros_joint_state_publisher.so">
+            <update_rate>20</update_rate>
+            <joint_name>front_left_wheel_joint</joint_name>
+            <joint_name>front_right_wheel_joint</joint_name>
+            <joint_name>back_left_wheel_joint</joint_name>
+            <joint_name>back_right_wheel_joint</joint_name>
+        </plugin>
+    </gazebo>
+    <!-- create link and joint for optical camera frame -->
+    <joint name="camera_optical_joint" type="fixed">
+        <origin xyz = "0 0 0" rpy="-1.571 0 -1.571"/>
+        <parent link="camera_link"/>
+        <child link="camera_link_opical"/>
+    </joint>
+    <link name="camera_link_optical"></link>
+    <!-- add gazebo setup for camera-->
+    <gazebo reference="camera_link">
+        <sensor type="depth" name="zed2i">
+            <update_rate>20</update_rate>
+            <visualize>true</visualize>
+            <camera name="zed">
+                <horizontal_fov>1.3962634</horizontal_fov>
+                <image>
+                    <width>640</width>
+                    <height>480</height>
+                    <format>R8B8G8</format>
+                </image>
+                <clip>
+                    <near>0.02</near>
+                    <far>300</far>
+                </clip>
+                <noise>
+                    <type>gaussian</type>
+                    <mean>0.0</mean>
+                    <stddev>0.007</stddev>
+                </noise>
+            </camera>
+            <plugin name="camera_controller" filename="libgazebo_ros_camera.so"
+        </sensor>
+    </gazebo>
 </robot>

File: helios/description/robot.urdf.xacro (robot description, xacro)
@@ -2,6 +2,6 @@
 <robot xmlns:xacro="http://www.ros.org/wiki/xacro" name="helios">
     <xacro:include filename="robot_core.xacro"/>
-    <xacro:include filename="ros2_control.xacro"/>
-    <!-- <xacro:include filename="gazebo.xacro"/>
-    <xacro:include filename="lidar.xacro"/> -->
+    <xacro:include filename="gazebo.xacro"/>
+    <!-- <xacro:include filename="ros2_control.xacro"/> -->
+    <!-- <xacro:include filename="lidar.xacro"/> -->
 </robot>

Commit message: colors added, joint states publishing, reformatted

File: helios/description/gazebo.xacro (robot description, xacro)
@@ -1,4 +1,19 @@
 <?xml version="1.0"?>
 <robot xmlns:xacro="http://www.ros.org/wiki/xacro">]
+    <gazebo reference="chassis">
+        <material>Gazebo/White</material>
+    </gazebo>
+    <gazebo reference="front_left_wheel">
+        <material>Gazebo/Blue</material>
+    </gazebo>
+        <gazebo reference="front_right_wheel">
+        <material>Gazebo/Blue</material>
+    </gazebo>
+        <gazebo reference="back_left_wheel">
+        <material>Gazebo/Blue</material>
+    </gazebo>
+        <gazebo reference="back_right_wheel">
+        <material>Gazebo/Blue</material>
+    </gazebo>
     <!-- TODO change later to use gazebo_ros_control plugin instead -->
     <gazebo>
@@ -13,12 +28,12 @@
     </gazebo>
     <!-- create link and joint for optical camera frame -->
-    <joint name="camera_optical_joint" type="fixed">
+    <!-- <joint name="camera_optical_joint" type="fixed">
         <origin xyz = "0 0 0" rpy="-1.571 0 -1.571"/>
         <parent link="camera_link"/>
         <child link="camera_link_opical"/>
     </joint>
-    <link name="camera_link_optical"></link>
+    <link name="camera_link_optical"></link> -->
     <!-- add gazebo setup for camera-->
-    <gazebo reference="camera_link">
+    <!-- <gazebo reference="camera_link">
         <sensor type="depth" name="zed2i">
             <update_rate>20</update_rate>
@@ -41,6 +56,6 @@
                 </noise>
             </camera>
-            <plugin name="camera_controller" filename="libgazebo_ros_camera.so"
+            <plugin name="camera_controller" filename="libgazebo_ros_camera.so">
         </sensor>
-    </gazebo>
+    </gazebo> -->
 </robot>

Commit message: Got lidar working.

File: helios/description/gazebo.xacro (robot description, xacro)
@@ -69,3 +69,44 @@
         </sensor>
     </gazebo>
+    <!-- Add gazebo setup for LIDAR -->
+    <!-- lidar -->
+    <gazebo reference="lidar_link">
+        <sensor type="gpu_ray" name="lidar">
+            <pose>0 0 0 0 0 0</pose>
+            <visualize>true</visualize>
+            <update_rate>40</update_rate>
+            <ray>
+                <scan>
+                    <horizontal>
+                        <samples>720</samples>
+                        <resolution>1</resolution>
+                        <min_angle>-1.570796</min_angle>
+                        <max_angle>1.570796</max_angle>
+                    </horizontal>
+                </scan>
+                <range>
+                    <min>0.10</min>
+                    <max>30.0</max>
+                    <resolution>0.01</resolution>
+                </range>
+                <noise>
+                    <type>gaussian</type>
+                    <!-- TODO - Add correct noise parameters for lidar specs - example is below. -->
+                    <!-- Noise parameters based on published spec for Hokuyo laser
+                        achieving "+-30mm" accuracy at range < 10m.  A mean of 0.0m and
+                        stddev of 0.01m will put 99.7% of samples within 0.03m of the true
+                        reading. -->
+                    <mean>0.0</mean>
+                    <stddev>0.01</stddev>
+                </noise>
+            </ray>
+            <plugin name="lidar_controller" filename="libgazebo_ros_ray_sensor.so">
+                <ros>
+                    <argument>~/out:=scan</argument>
+                </ros>
+                <output_type>sensor_msgs/LaserScan</output_type>
+                <frameName>lidar_link</frameName>
+            </plugin>
+        </sensor>
+    </gazebo>
 </robot>

File: helios/description/sensors.xacro (robot description, xacro)
@@ -57,3 +57,32 @@
         </xacro:inertial_box>
     </link>
+    <!-- LIDAR  -->
+    <!-- Lidar Joint -->
+    <joint name="lidar_joint" type="fixed">
+        <axis xyz="0 1 0" />
+        <origin xyz="0 3 0" rpy="0 0 0"/>
+        <parent link="chassis_link"/>
+        <child link="lidar_link"/>
+    </joint>
+    <!-- Lidar Link -->
+    <link name="lidar_link">
+        <collision>
+            <origin xyz="0 0 0" rpy="0 0 0"/>
+            <geometry>
+                <box size="0.1 0.1 0.1"/>
+            </geometry>
+        </collision>
+        <visual>
+            <origin xyz="0 0 0" rpy="0 0 0"/>
+            <geometry>
+                <box size="0.1 0.1 0.1"/>
+            </geometry>
+        </visual>
+        <!-- ToDO replace this -->
+        <inertial>
+            <mass value="1e-5" />
+            <origin xyz="0 0 0" rpy="0 0 0"/>
+            <inertia ixx="1e-6" ixy="0" ixz="0" iyy="1e-6" iyz="0" izz="1e-6" />
+        </inertial>
+    </link>
 </robot>

Commit message: Fixed lidar positioning

File: helios/description/gazebo.xacro (robot description, xacro)
@@ -72,5 +72,5 @@
     <!-- lidar -->
     <gazebo reference="lidar_link">
-        <sensor type="gpu_ray" name="lidar">
+        <sensor type="gpu_ray" name="lidar"> <!-- "gpu_ray" to use GPU, "ray" to use CPU -->
             <pose>0 0 0 0 0 0</pose>
             <visualize>true</visualize>
@@ -86,6 +86,6 @@
                 </scan>
                 <range>
-                    <min>0.10</min>
-                    <max>30.0</max>
+                    <min>0.2</min>
+                    <max>16</max>
                     <resolution>0.01</resolution>
                 </range>
@@ -102,7 +102,5 @@
             </ray>
             <plugin name="lidar_controller" filename="libgazebo_ros_ray_sensor.so">
-                <ros>
-                    <argument>~/out:=scan</argument>
-                </ros>
+                <topicName>/lidar/scan</topicName>
                 <output_type>sensor_msgs/LaserScan</output_type>
                 <frameName>lidar_link</frameName>

File: helios/description/sensors.xacro (robot description, xacro)
@@ -70,5 +70,5 @@
     <joint name="lidar_joint" type="fixed">
         <axis xyz="0 1 0" />
-        <origin xyz="0 0 1" rpy="0 0 0"/>
+        <origin xyz="0.7 0 0.24" rpy="0 0 0"/>
         <parent link="chassis_link"/>
         <child link="lidar_link"/>

Commit message: Added correct property values for lidar

File: helios/description/gazebo.xacro (robot description, xacro)
@@ -22,4 +22,7 @@
         <material>Gazebo/Black</material>
     </gazebo>
+    <gazebo reference="lidar_link">
+        <material>Gazebo/Grey</material>
+    </gazebo>
     <!-- TODO change later to use gazebo_ros_control plugin instead -->
     <gazebo>
@@ -40,5 +43,5 @@
     </joint>
     <link name="zed2i_link_optical"></link>
-    <!-- add gazebo setup for camera-->
+    <!-- Gazebo setup for camera-->
     <gazebo reference="zed2i_link">
         <sensor type="camera" name="zed2i">
@@ -69,6 +72,5 @@
         </sensor>
     </gazebo>
-    <!-- Add gazebo setup for LIDAR -->
-    <!-- lidar -->
+    <!-- Gazebo setup for LIDAR -->
     <gazebo reference="lidar_link">
         <sensor type="gpu_ray" name="lidar"> <!-- "gpu_ray" to use GPU, "ray" to use CPU -->
@@ -81,6 +83,6 @@
                         <samples>720</samples>
                         <resolution>1</resolution>
-                        <min_angle>-1.570796</min_angle>
-                        <max_angle>1.570796</max_angle>
+                        <min_angle>-2.35619</min_angle>
+                        <max_angle>2.35619</max_angle>
                     </horizontal>
                 </scan>
@@ -102,5 +104,4 @@
             </ray>
             <plugin name="lidar_controller" filename="libgazebo_ros_ray_sensor.so">
-                <topicName>/lidar/scan</topicName>
                 <output_type>sensor_msgs/LaserScan</output_type>
                 <frameName>lidar_link</frameName>

File: helios/description/sensors.xacro (robot description, xacro)
@@ -62,13 +62,12 @@
     </link>
     <!-- LIDAR ======================================================== -->
-    <!-- TODO - Update property values to be correct -->
     <!-- LIDAR Properties -->
-    <xacro:property name="lidar_height" value="0.03"/>
-    <xacro:property name="lidar_radius" value="0.03"/>
-    <xacro:property name="lidar_mass" value="0.01"/>
+    <xacro:property name="lidar_height" value="0.041"/>
+    <xacro:property name="lidar_radius" value="0.038"/>
+    <xacro:property name="lidar_mass" value="0.19"/>
     <!-- LIDAR Joint -->
     <joint name="lidar_joint" type="fixed">
         <axis xyz="0 1 0" />
-        <origin xyz="0.7 0 0.24" rpy="0 0 0"/>
+        <origin xyz="0.9 0 0.25" rpy="0 0 0"/>
         <parent link="chassis_link"/>
         <child link="lidar_link"/>

Commit message: Began Adding IMU stuff

File: helios/description/gazebo.xacro (robot description, xacro)
@@ -23,4 +23,7 @@
     </gazebo>
     <gazebo reference="lidar_link">
+        <material>Gazebo/Grey</material>
+    </gazebo>
+    <gazebo reference="imu_link">
         <material>Gazebo/Grey</material>
     </gazebo>
@@ -103,5 +106,5 @@
                 </noise>
             </ray>
-            <plugin name="lidar_controller" filename="libgazebo_ros_ray_sensor.so">
+            <plugin name="lidar_plugin" filename="libgazebo_ros_ray_sensor.so">
                 <output_type>sensor_msgs/LaserScan</output_type>
                 <frameName>lidar_link</frameName>
@@ -109,3 +112,24 @@
         </sensor>
     </gazebo>
+    <!-- Gazebo setup for IMU -->
+    <gazebo reference="imu_link">
+    <gravity>true</gravity>
+    <sensor name="imu_sensor" type="imu">
+        <always_on>true</always_on>
+        <update_rate>100</update_rate>
+        <visualize>true</visualize>
+        <topic>__default_topic__</topic>
+        <plugin filename="libgazebo_ros_imu_sensor.so" name="imu_plugin">
+            <topicName>imu</topicName>
+            <bodyName>imu_link</bodyName>
+            <updateRateHZ>10.0</updateRateHZ>
+            <gaussianNoise>0.0</gaussianNoise>
+            <xyzOffset>0 0 0</xyzOffset>
+            <rpyOffset>0 0 0</rpyOffset>
+            <frameName>imu_link</frameName>
+            <initialOrientationAsReference>false</initialOrientationAsReference>
+        </plugin>
+        <pose>0 0 0 0 0 0</pose>
+    </sensor>
+    </gazebo>
 </robot>

File: helios/description/sensors.xacro (robot description, xacro)
@@ -75,10 +75,10 @@
     <!-- LIDAR Link -->
     <link name="lidar_link">
-        <collision>
+        <!-- <collision>
             <origin xyz="0 0 0" rpy="0 0 0"/>
             <geometry>
                 <cylinder length="${lidar_height}" radius="${lidar_radius}"/>
             </geometry>
-        </collision>
+        </collision> -->
         <visual>
             <origin xyz="0 0 0" rpy="0 0 0"/>
@@ -91,3 +91,33 @@
         </xacro:inertial_cylinder>
     </link>
+    <!-- TODO - Get correct property values -->
+    <!-- NavX ======================================================== -->
+    <!-- NavX -->
+    <!-- <xacro:property name="navx_height" value="0.041"/>
+    <xacro:property name="navx_radius" value="0.038"/> -->
+    <!-- NavX Joint -->
+    <joint name="navx_joint" type="fixed">
+        <axis xyz="0 1 0" />
+        <origin xyz="0.5 0 0.25" rpy="0 0 0"/>
+        <parent link="chassis_link"/>
+        <child link="navx_link"/>
+    </joint>
+    <!-- NavX Link -->
+    <link name="navx_link">
+        <!-- <collision>
+            <origin xyz="0 0 0" rpy="0 0 0"/>
+            <geometry>
+                <cylinder length="${navx_height}" radius="${navx_radius}"/>
+            </geometry>
+        </collision> -->
+        <!-- <visual>
+            <origin xyz="0 0 0" rpy="0 0 0"/>
+            <geometry>
+                <cylinder length="${navx_height}" radius="${navx_radius}"/>
+            </geometry>
+        </visual> -->
+        <!-- <xacro:inertial_cylinder mass="${navx_mass}" length="${navx_height}" radius="${navx_radius}">
+            <origin xyz="0 0 0" rpy="0 0 0"/>
+        </xacro:inertial_cylinder> -->
+    </link>
 </robot>
